File: airmed_board_v1.0/airmed_board_v1.0.sch (KiCad schematic (older format))
At the start: 31 parts, among them J1 Barrel_Jack, J2 Conn_01x03_Female, J3 Conn_01x05_Female, J4 Conn_01x09_Female, J5 Conn_01x08_Female, Q1 Q_NMOS_DGS, U1 LD1117S50TR_SOT223, U2 LD1117S33TR_SOT223, U3 CC3220, U4 74HC4051, U5 74HC4051

Commit message: Board Schematic v1.0 updated
Parts:
- removed BZ1: Buzzer, symbol Device:Buzzer
- removed J2: Conn_01x03_Female, symbol Connector:Conn_01x03_Female
- removed J3: Conn_01x05_Female, symbol Connector:Conn_01x05_Female
- removed J4: Conn_01x09_Female, symbol Connector:Conn_01x09_Female
- removed J5: Conn_01x08_Female, symbol Connector:Conn_01x08_Female
- removed Q1: Q_NMOS_DGS, symbol Device:Q_NMOS_DGS
- removed R10, R11, R8, R9: 100, symbol Device:R
- removed R12, R13: 1M, symbol Device:R
- removed U4, U5: 74HC4051, symbol 74xx:74HC4051
- added AE1: Antenna_Shield, RF_Antenna:AH316M, symbol Device:Antenna_Shield
- added C10, C15, C9: 10u, Capacitor_SMD:C_0603_1608Metric, symbol Device:C
- added C11, C13, C14, C16, C17, C18, C19, C20, C21: 0.1u, Capacitor_SMD:C_0402_1005Metric, symbol Device:C
- added C12, C7, C8: 4.7u, Capacitor_SMD:C_0402_1005Metric, symbol Device:C
- added C22, C24: 6.2p, Capacitor_SMD:C_0402_1005Metric, symbol Device:C
- added C23: 0.1uF, Capacitor_SMD:C_0402_1005Metric, symbol Device:C
- added C25, C27: 10p, Capacitor_SMD:C_0402_1005Metric, symbol Device:C
- added C26, C28: 0.5p, Capacitor_SMD:C_0402_1005Metric, symbol Device:C
- added J2: Conn_02x03_Odd_Even, Connector_PinHeader_2.54mm:PinHeader_2x03_P2.54mm_Vertical, symbol Connector_Generic:Conn_02x03_Odd_Even
- added J3: Conn_01x21_Female, Connector_PinSocket_2.54mm:PinSocket_1x21_P2.54mm_Vertical, symbol Connector:Conn_01x21_Female
- added J5: Conn_02x05_Odd_Even, Connector_PinHeader_1.27mm:PinHeader_2x05_P1.27mm_Vertical_SMD, symbol Connector_Generic:Conn_02x05_Odd_Even
- added L1, L3: 2.2uH, Inductor_SMD:L_1206_3216Metric, symbol Device:L
- added L2: 1uH, Inductor_SMD:L_1206_3216Metric, symbol Device:L
- added L4: 10uH, Inductor_SMD:L_1206_3216Metric, symbol Device:L
- added L5, L6: 3.3nH, Inductor_SMD:L_0402_1005Metric, symbol Device:L
- added SW1: SW_SPDT, Button_Switch_THT:SW_CuK_OS102011MA1QN1_SPDT_Angled, symbol Switch:SW_SPDT
- added U4: DEA202450BT-1294C1-H, Filter:TDKFilter1294C1H, symbol Device:DEA202450BT-1294C1-H
- added U5: MX25R3235F, Package_SO:SSOP-8_3.9x5.05mm_P1.27mm, symbol Memory_Flash:MX25R3235F
- added Y1: Crystal_GND24, Crystal:Crystal_SMD_Epson_FA-20H-4pin_2.5mm_2.0mm, symbol Device:Crystal_GND24
- added Y2: Crystal, Crystal:Crystal_SMD_Abracon_ABS07-2Pin_3.2mm_1.5mm, symbol Device:Crystal
- C1: value 10u -> 22u; footprint (none) -> Capacitor_SMD:C_0603_1608Metric
- C2: value 100n -> 22u; footprint (none) -> Capacitor_SMD:C_0603_1608Metric
- C3: value 10n -> 0.1uF; footprint (none) -> Capacitor_SMD:C_0402_1005Metric
- C4, C5: footprint (none) -> Capacitor_SMD:C_0603_1608Metric
- C6: footprint (none) -> Capacitor_SMD:C_0402_1005Metric
- J1: footprint (none) -> Connector_BarrelJack:BarrelJack_CUI_PJ-063AH_Horizontal
- R1, R3, R5: value 1M -> 100k; footprint (none) -> Resistor_SMD:R_0402_1005Metric
- R2: value 1M -> 0; footprint (none) -> Resistor_SMD:R_0402_1005Metric
- R4: value 1M -> 2.7k; footprint (none) -> Resistor_SMD:R_0402_1005Metric
- R6: value 2.2k -> 100K; footprint (none) -> Resistor_SMD:R_0402_1005Metric
- R7: value 1M -> 1K; footprint (none) -> Resistor_SMD:R_0402_1005Metric
- U1: value LD1117S50TR_SOT223 -> AP1084K50L-13; footprint Package_TO_SOT_SMD:SOT-223-3_TabPin2 -> Package_TO_SOT_SMD:TO-263-2
- U2: value LD1117S33TR_SOT223 -> AZ1084CD-3.3TRG1; footprint Package_TO_SOT_SMD:SOT-223-3_TabPin2 -> Package_TO_SOT_SMD:TO-252-2
- U3: footprint (none) -> TI_MCU:CC3220; symbol MCU_Texas:CC3220 -> airmed_board_v1.0-rescue:CC3220-MCU_Texas
Connections:
- net BEAM_4 is gone; now on net TCK: U3.19 (TCK)
- net +12V: no longer C1.1, C2.1
- net +3V3: now also R2.2, R6.1, R7.2, C12.1, C18.1, C20.1, C23.1, C7.1, C8.1, J2.2 (Pin_2), J2.4 (Pin_4), J2.6 (Pin_6), U5.3 (WP#/SIO2), U5.7 (RESET#/SIO3), U5.8 (VCC); no longer C6.2, R6.2
- net GND: now also C6.2, U3.GND_TAB (65), AE1.1 (A), AE1.2 (Shield), C10.2, C11.2, C12.2, C13.2, C14.2, C15.2, C16.2, C17.2, C18.2, C19.2, C20.2, C21.2, C22.2, C23.2, C24.2, C25.2, C26.1, C26.2, C27.2, C28.1, C28.2, C7.2, C8.2, C9.2, J5.3 (Pin_3), J5.5 (Pin_5), J5.7 (Pin_7), J5.9 (Pin_9), L5.2, L6.2, U4.2 (GND), U4.4 (GND), U5.4 (GND), Y1.2, Y1.4; no longer R2.2, R7.2
- net at U3.11 (FLASH_SPI_CLK): now also U5.6 (SCLK)
- net at U3.12 (FLASH_SPI_DOUT): now also U5.5 (SI?SIO0)
- net at U3.13 (FLASH_SPI_DIN): now also U5.2 (SI/SIO1)
- net at U3.14 (FLASH_SPI_CS): now also R6.2, U5.1 (CS#)
- net at U3.21 (SPO2): now also R4.1, J2.5 (Pin_5)
- net at U3.22 (WLAN_XTAL_N): now also C22.1, Y1.1
- net at U3.23 (WLAN_XTAL_P): now also C24.1, Y1.3
- net at U3.24 (VDD_PLL): now also C21.1
- net at U3.25 (LDO_IN2): now also U3.36 (LDO_IN1), U3.48 (VDD_ANA1), C11.1, C14.1, C17.1, C9.1, L1.1
- net at U3.31 (RF_BG): now also U4.1 (In)
- net nRESET: now reaches U3.32 (nRESET)
- net nRESET: now also J5.10 (Pin_10)
- net at U3.33 (CDD_PA_IN): now also C1.1, C2.1, C6.1, U3.42 (DCDC_PA_OUT)
- net at U3.34 (SOP1): now also R3.1, J2.3 (Pin_3)
- net at U3.35 (SOP0): now also R1.1, J2.1 (Pin_1)
- net at U3.38 (DCDC_ANA_SW): now also L1.2
- net at U3.40 (DCDC_PA_SW_P): now also L2.2
- net at U3.41 (DCDC_PA_SW_N): now also L2.1
- net at U3.43 (DCDC_DIG_SW): now also L3.2
- net at U3.46 (DCDC_ANA2_SW_N): now also L4.1
- net at U3.47 (VDD_ANA2): now also R2.1, C15.1
- net at U3.49 (VDD_RAM): now also C19.1
- net at U3.51 (RTC_XTAL_P): now also C27.1, Y2.2
- net at U3.52 (RTC_XTAL_N): now also C25.1, Y2.1
- net at U3.56 (VDD_DIG2): now also U3.9 (VDD_DIG1), C10.1, C13.1, C16.1, L3.1
- net at U3.60 (GPIO5): now also J3.6 (Pin_6)
- net at R7.1: now also J5.1 (Pin_1)
- net TCK: now reaches R5.1
- net TCK: now also J5.4 (Pin_4)
- net BEAM_1 renamed TDI
- net TDI: now also J5.8 (Pin_8)
- net BEAM_2 renamed TDO
- net TDO: now also J5.6 (Pin_6)
- net BEAM_3: no longer names the net of U3.18 (GPIO28)
- net BEAM_3: now also J3.20 (Pin_20)
- net BEAM_5 renamed TMS
- net TMS: now also J5.2 (Pin_2)
- net BEAM_6: no longer names the net of U3.45 (DCDC_ANA2_SW_P)
- net BEAM_6: now also L4.2
- net BEAM_7: no longer names the net of U3.58 (GPIO3)
- net BEAM_7: now also J3.4 (Pin_4)
- net BEAM_8: no longer names the net of U3.59 (GPIO4)
- net BEAM_8: now also J3.5 (Pin_5)
- net BUZZER: no longer names the net of U3.15 (GPIO22)
- net BUZZER: now also J3.19 (Pin_19)
- net LED_1: no longer names the net of U3.50 (GPIO0)
- net LED_1: now also J3.1 (Pin_1)
- net LED_2: no longer names the net of U3.53 (GPIO30)
- net LED_2: now also J3.21 (Pin_21)
- net LED_3: no longer names the net of U3.55 (GPIO1)
- net LED_3: now also J3.2 (Pin_2)
- net LED_4: no longer names the net of U3.57 (GPIO2)
- net LED_4: now also J3.3 (Pin_3)
- net MOTOR_CTRL_A: no longer names the net of U3.2 (GPIO11)
- net MOTOR_CTRL_A: now also J3.12 (Pin_12)
- net MOTOR_CTRL_B: no longer names the net of U3.3 (GPIO12)
- net MOTOR_CTRL_B: now also J3.13 (Pin_13)
- net MOTOR_CTRL_C: no longer names the net of U3.4 (GPIO13)
- net MOTOR_CTRL_C: now also J3.14 (Pin_14)
- net MOTOR_CTRL_D: no longer names the net of U3.5 (GPIO14)
- net MOTOR_CTRL_D: now also J3.15 (Pin_15)
- net MOTOR_CTRL_E: no longer names the net of U3.61 (GPIO6)
- net MOTOR_CTRL_E: now also J3.7 (Pin_7)
- net MOTOR_CTRL_F: no longer names the net of U3.62 (GPIO7)
- net MOTOR_CTRL_F: now also J3.8 (Pin_8)
- net MOTOR_CTRL_G: no longer names the net of U3.63 (GPIO8)
- net MOTOR_CTRL_G: now also J3.9 (Pin_9)
- net MOTOR_CTRL_H: no longer names the net of U3.64 (GPIO9)
- net MOTOR_CTRL_H: now also J3.10 (Pin_10)
- net SERVO_PWM: no longer names the net of U3.1 (GPIO10)
- net SERVO_PWM: now also J3.11 (Pin_11)
- net SERVO_SEL_1: no longer names the net of U3.6 (GPIO15)
- net SERVO_SEL_1: now also J3.16 (Pin_16)
- net SERVO_SEL_2: no longer names the net of U3.7 (GPIO16)
- net SERVO_SEL_2: now also J3.17 (Pin_17)
- net SERVO_SEL_3: no longer names the net of U3.8 (GPIO17)
- net SERVO_SEL_3: now also J3.18 (Pin_18)
- new net: L5.1, SW1.1 (A)
- new net: SW1.2 (B), U4.3 (Out)
- new net: L6.1, SW1.3 (C)
- no-connect marks 31 -> 2
Other:
- note added: "1 of 1"
- note added: "Apotech Board V1.0"
- note added: "October, 31 2018"
- note added: "Version History:\nCreated: Oct 14, 2018\nRelease A: Oct 31, 2018\n"
- note added: "airmed_board_v1.0.esh"
- moved on the sheet: C3, C4, C5, J1, U1, U2
