File: airmed_board_v1.0/motor_drivers.sch (KiCad schematic (older format))
At the start: 20 parts, among them J6 Conn_01x16_Female, U10 74LS14, U11 SN754410, U12 SN754410, U6 74LS14, U7 74LS14, U8 SN754410, U9 SN754410

Commit message: Board Schematic v1.0 updated
Parts:
- removed R15, R16, R17: R, symbol Device:R
- removed U10, U6, U7: 74LS14, symbol 74xx:74LS14
- removed U11, U12, U9: SN754410, symbol Driver_Motor:SN754410
- added R1, R2, R3: 10k, symbol Device:R
- added U6, U7, U9: SN754410, symbol airmed_board_v1.0-rescue:SN754410-Driver_Motor
- R14: value R -> 10k
- U8: symbol Driver_Motor:SN754410 -> airmed_board_v1.0-rescue:SN754410-Driver_Motor
Connections:
- net +12V: now also U6.8 (Vcc2), U7.8 (Vcc2), U9.8 (Vcc2)
- net +5V: now also R1.2, R2.2, R3.2, U6.16 (Vcc1), U7.16 (Vcc1), U9.16 (Vcc1)
- net GND: now also U6.12 (Ground), U6.13 (Ground), U6.4 (Ground), U6.5 (Ground), U7.12 (Ground), U7.13 (Ground), U7.4 (Ground), U7.5 (Ground), U9.12 (Ground), U9.13 (Ground), U9.4 (Ground), U9.5 (Ground)
- net MOTOR_A_N: now also U8.6 (Output2)
- net MOTOR_A_P: now also U8.3 (Output1)
- net MOTOR_B_N: now also U8.14 (Output4)
- net MOTOR_B_P: now also U8.11 (Output3)
- net MOTOR_C_N: now also U9.6 (Output2); no longer U8.6 (Output2)
- net MOTOR_C_P: now also U9.3 (Output1); no longer U8.3 (Output1)
- net MOTOR_D_N: now also U9.14 (Output4); no longer U8.14 (Output4)
- net MOTOR_D_P: now also U9.11 (Output3); no longer U8.11 (Output3)
- net MOTOR_E_N: now also U6.6 (Output2)
- net MOTOR_E_P: now also U6.3 (Output1)
- net MOTOR_F_N: now also U6.14 (Output4)
- net MOTOR_F_P: now also U6.11 (Output3)
- net MOTOR_G_N: now also U7.6 (Output2)
- net MOTOR_G_P: now also U7.3 (Output1)
- net MOTOR_H_N: now also U7.14 (Output4)
- net MOTOR_H_P: now also U7.11 (Output3)
- net at C11.1: now also R2.1, U7.1 (1,2Enable), U7.9 (3,4Enable)
- net MOTOR_CTRL_B_P: now reaches U8.10 (Input3)
- net MOTOR_CTRL_B_N: now reaches U8.15 (Input4)
- net MOTOR_CTRL_A_P: now reaches U8.2 (Input1)
- net MOTOR_CTRL_A_N: now reaches U8.7 (Input2)
- net at C12.1: now also R3.1, U9.1 (1,2Enable), U9.9 (3,4Enable)
- net at C8.1: now also R1.1, U6.1 (1,2Enable), U6.9 (3,4Enable)
- new net MOTOR_CTRL_C_N: U9.7 (Input2)
- new net MOTOR_CTRL_C_P: U9.2 (Input1)
- new net MOTOR_CTRL_D_N: U9.15 (Input4)
- new net MOTOR_CTRL_D_P: U9.10 (Input3)
- new net MOTOR_CTRL_E_N: U6.7 (Input2)
- new net MOTOR_CTRL_E_P: U6.2 (Input1)
- new net MOTOR_CTRL_F_N: U6.15 (Input4)
- new net MOTOR_CTRL_F_P: U6.10 (Input3)
- new net MOTOR_CTRL_G_N: U7.7 (Input2)
- new net MOTOR_CTRL_G_P: U7.2 (Input1)
- new net MOTOR_CTRL_H_N: U7.15 (Input4)
- new net MOTOR_CTRL_H_P: U7.10 (Input3)
Other:
- moved on the sheet: C7, C9, R14, U8
