File: airmed_board_v1.0/_saved_airmed_board_v1.0.sch (KiCad schematic (older format))
At the start: 57 parts, among them J1 Barrel_Jack, J2 Conn_02x03_Odd_Even, J3 Conn_02x15_Top_Bottom, J5 Conn_02x05_Odd_Even, SW1 SW_SPDT, SW2 SW_Push, U1 AP1084K50L-13, U2 AZ1084CD-3.3TRG1, U3 CC3220, U4 DEA202450BT-1294C1-H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

Commit message: board
Parts:
- J1: footprint Connector_BarrelJack:BarrelJack_CUI_PJ-063AH_Horizontal -> Connector_BarrelJack:BarrelJack_CUI_PJ-037A_Horizontal
Changed lines of the file:
@@
 F 0 "J1" V 1000 5800 50  0000 L CNN
 F 1 "Barrel_Jack" V 1100 5550 50  0000 L CNN
-F 2 "Connector_BarrelJack:BarrelJack_CUI_PJ-063AH_Horizontal" H 1050 6110 50  0001 C CNN
+F 2 "Connector_BarrelJack:BarrelJack_CUI_PJ-037A_Horizontal" H 1050 6110 50  0001 C CNN
 F 3 "https://www.cui.com/product/resource/pj-037a.pdf" H 1050 6110 50  0001 C CNN
 	1    1000 6150
