File: airmed_board_w1.0/airmed_board_w1.0/airmed_board_w1.0.kicad_pcb (KiCad board)
At the start: 2 copper layers, 62.2 x 41.4 mm, 53 parts, among them IC1 CC3220MODASF12MONR, IC2 MX25R3235FM1IL0, J1 Conn_01x03_Male, J2 Barrel_Jack, J3 Conn_02x03_Odd_Even, J4 Conn_02x05_Odd_Even, J5 Conn_02x15_Odd_Even, Q1 Q_NMOS_GSD, Q2 Q_NMOS_GSD, Q3 Q_NMOS_GSD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

Commit message: added literally everything
Other:
- rule pad_to_mask_clearance: 0.051 -> 0.005
- rule solder_mask_min_width: 0.25 -> 0.1
Changed lines of the file:
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@@
     (pad_size 0.75 0.3)
     (pad_drill 0)
-    (pad_to_mask_clearance 0.051)
-    (solder_mask_min_width 0.25)
+    (pad_to_mask_clearance 0.005)
+    (solder_mask_min_width 0.1)
     (aux_axis_origin 0 0)
     (visible_elements FFFFFF7F)
@@
       (creategerberjobfile false)
       (excludeedgelayer false)
-      (linewidth 0.100000)
+      (linewidth 0.020000)
       (plotframeref false)
       (viasonmask false)
